Commit message: daily backup: 2026-08-12 17:00 Asia/Shanghai

File: src/xw_description/urdf/xw_gen2.urdf (robot description, URDF)
Before this commit: robot xw_gen2, 5 links, 4 joints
Links:
- added link camera_front_2_link
- added link imu_link
Joints:
- added joint camera_front_2_joint: type fixed, parent base_link, child camera_front_2_link, origin xyz=0.18 0 0.28 rpy=-1.1 0 -1.5708
- added joint imu_joint: type fixed, parent base_link, child imu_link, origin xyz=0 0 0.10 rpy=0 0 0
- joint camera_front_joint: origin xyz=0.18 0 0.25 rpy=0 0 0 -> xyz=0.18 0 0.25 rpy=-1.3955 0 -1.5708

Commit message: daily backup: 2026-08-13 17:00 Asia/Shanghai

File: src/xw_description/urdf/xw_gen2.urdf (robot description, URDF)
Before this commit: robot xw_gen2, 7 links, 6 joints
Links:
- removed link camera_front_2_link
- removed link camera_front_link
- added link camera_front_down_link
- added link camera_front_up_link
Joints:
- removed joint camera_front_2_joint
- removed joint camera_front_joint
- added joint camera_front_down_joint: type fixed, parent base_link, child camera_front_down_link, origin xyz=0.18 0 0.28 rpy=-1.1 0 -1.5708
- added joint camera_front_up_joint: type fixed, parent base_link, child camera_front_up_link, origin xyz=0.18 0 0.25 rpy=-1.3955 0 -1.5708
- joint lidar_joint: origin xyz=0 0 0.22 rpy=0 0 0 -> xyz=0 0 0.22 rpy=0 0 3.141592653589793

Commit message: auto-sync: 2026-08-19 05:42:10 [docker-manual]

File: src/xw_description/urdf/xw_gen2.urdf (robot description, URDF)
Before this commit: robot xw_gen2, 7 links, 6 joints
Joints:
- joint camera_front_down_joint: origin xyz=0.18 0 0.28 rpy=-1.1 0 -1.5708 -> xyz=0.18 0 0.25 rpy=-1.1 0 -1.5708
- joint camera_front_up_joint: origin xyz=0.18 0 0.25 rpy=-1.3955 0 -1.5708 -> xyz=0.18 0 0.28 rpy=-1.3955 0 -1.5708

Commit message: daily backup: 2026-08-31 17:00 Asia/Shanghai

File: src/xw_description/urdf/xw_gen2.urdf (robot description, URDF)
Before this commit: robot xw_gen2, 7 links, 6 joints
Joints:
- joint camera_front_down_joint: origin xyz=0.18 0 0.25 rpy=-1.1 0 -1.5708 -> xyz=0.251 0 0.16 rpy=-0.895 0 -1.5708
- joint camera_front_up_joint: origin xyz=0.18 0 0.28 rpy=-1.3955 0 -1.5708 -> xyz=0.251 0 0.49 rpy=-2.181 0 -1.5708
- joint imu_joint: origin xyz=0 0 0.10 rpy=0 0 0 -> xyz=0 0 0.37 rpy=0 0 0
- joint lidar_joint: origin xyz=0 0 0.22 rpy=0 0 3.141592653589793 -> xyz=0 0 0.10 rpy=0 0 3.141592653589793

Commit message: daily backup: 2026-08-31 17:00 Asia/Shanghai

File: src/xw_description/urdf/xw_gen2.urdf (robot description, URDF)
Before this commit: robot xw_gen2, 7 links, 6 joints
Joints:
- joint camera_front_down_joint: origin xyz=0.251 0 0.16 rpy=-0.895 0 -1.5708 -> xyz=0.251 0 0.16 rpy=-1.09 0 -1.5708

Commit message: daily backup: 2026-09-03 17:00 Asia/Shanghai

File: src/xw_description/urdf/xw_gen2.urdf (robot description, URDF)
Before this commit: robot xw_gen2, 7 links, 6 joints
Joints:
- joint camera_front_down_joint: origin xyz=0.251 0 0.16 rpy=-1.09 0 -1.5708 -> xyz=0.251 0 0.16 rpy=-1.64 0 -1.5708
- joint camera_front_up_joint: origin xyz=0.251 0 0.49 rpy=-2.181 0 -1.5708 -> xyz=0.251 0 0.49 rpy=-1.64 0 -1.5708

Commit message: daily backup: 2026-09-03 17:00 Asia/Shanghai

File: src/xw_description/urdf/xw_gen2.urdf (robot description, URDF)
Before this commit: robot xw_gen2, 7 links, 6 joints
Joints:
- joint camera_front_up_joint: origin xyz=0.251 0 0.49 rpy=-1.64 0 -1.5708 -> xyz=0.251 0 0.49 rpy=-1.48 0 -1.5708

Commit message: daily backup: 2026-09-04 17:00 Asia/Shanghai

File: src/xw_description/urdf/xw_gen2.urdf (robot description, URDF)
Before this commit: robot xw_gen2, 7 links, 6 joints
Joints:
- joint camera_front_down_joint: origin xyz=0.251 0 0.16 rpy=-1.64 0 -1.5708 -> xyz=0.251 0 0.16 rpy=-2.01 0 -1.5708
- joint camera_front_up_joint: origin xyz=0.251 0 0.49 rpy=-1.48 0 -1.5708 -> xyz=0.251 0 0.49 rpy=-1.33 0 -1.5708

Commit message: daily backup: 2026-09-15 17:00 Asia/Shanghai

File: src/xw_description/urdf/xw_gen2.urdf (robot description, URDF)
Before this commit: robot xw_gen2, 7 links, 6 joints
Joints:
- joint camera_front_down_joint: origin xyz=0.251 0 0.16 rpy=-2.01 0 -1.5708 -> xyz=0.251 0 0.16 rpy=-2.04 0 -1.5708
- joint camera_front_up_joint: origin xyz=0.251 0 0.49 rpy=-1.33 0 -1.5708 -> xyz=0.251 0 0.49 rpy=-1.46 0 -1.5708
